File: nfc.kicad_sch (KiCad schematic)
At the start: 39 parts, among them U6 PN7160A1HN/C100E, Y1 27.12MHz / CL TBD

Commit message: Add PCB NFC coil and refine prototype component selections
Integrate a reusable 40 mm four-turn antenna footprint, calculated matching
network, hand-solder tuning pads, and a fabrication-ready bare-coil coupon.
Archive RF calculations, simulation results, reference sources, and tuning
instructions.

Select the PN7160 crystal and supply capacitors using manufacturer guidance
and DC-bias data. Record the confirmed 26-contact OLED interface and dedicated
5 V / 1.5 A USB-C source, retaining the JST-PH battery connector and deferred
battery behavior. Update the BOM, schematic PDFs, and verification tools.

Validation: native KiCad ERC reports zero violations; all current schematic
hashes match the verification report. Coil geometry, coupon DRC, RF model,
and component calculation results are archived with the design.
Parts:
- removed A1: 13.56MHz coil / TBD, Nucula_Project:NFC_Antenna_Interface_TBD, symbol Nucula_Project:NFC_Loop_TBD
- added A1: PCB loop 40x40 / 4T, Nucula_Project:NFC_PCB_Loop_40x40_4T_W0.50_S0.30, symbol Nucula_Project:NFC_PCB_Loop_40x40_4T
- added C53, C54: TRIM, Nucula_Project:C_0805_HandSolder_NoPaste, symbol Device:C
- added R41, R42: 0R, Resistor_SMD:R_0805_2012Metric_Pad1.20x1.40mm_HandSolder, symbol Device:R
- C15: LCSC (none) -> C28323; MPN (none) -> CL21B105KBFNNNE; Manufacturer (none) -> Samsung Electro-Mechanics; Placement (none) -> At U6.6 VDD_PAD; Tolerance 20% -> 10%; Voltage 10 V -> 50 V
- C16, C18, C20, C25: LCSC (none) -> C1591; MPN (none) -> CL10B104KB8NNNC; Manufacturer (none) -> Samsung Electro-Mechanics; Voltage 10 V -> 50 V
- C17: footprint Capacitor_SMD:C_0805_2012Metric -> Capacitor_SMD:C_1206_3216Metric; LCSC (none) -> C14860; MPN (none) -> CL31B106KAHNNNE; Manufacturer (none) -> Samsung Electro-Mechanics; Placement (none) -> At U6.12/28 VBAT; Tolerance 20% -> 10%; Voltage 10 V -> 25 V
- C19: footprint Capacitor_SMD:C_0805_2012Metric -> Capacitor_SMD:C_1206_3216Metric; LCSC (none) -> C14860; MPN (none) -> CL31B106KAHNNNE; Manufacturer (none) -> Samsung Electro-Mechanics; Placement (none) -> At U6.13 VDD_UP; Tolerance 20% -> 10%; Voltage 10 V -> 25 V
- C21: value 10uF -> 2.2uF; LCSC (none) -> C19110; MPN (none) -> CL21B225KAFNNNE; Manufacturer (none) -> Samsung Electro-Mechanics; Placement (none) -> Local capacitor at U6.26 VDDA; Status (none) -> PN7160 AN12988 local decoupling; selected stocked prototype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; Tolerance 20% -> 10%; Voltage 10 V -> 25 V
- C22: value 100nF -> 2.2uF; footprint Capacitor_SMD:C_0603_1608Metric -> Capacitor_SMD:C_0805_2012Metric; LCSC (none) -> C19110; MPN (none) -> CL21B225KAFNNNE; Manufacturer (none) -> Samsung Electro-Mechanics; Placement (none) -> Local capacitor at U6.27 VDD; Status (none) -> PN7160 AN12988 local decoupling; selected stocked prototype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; Voltage 10 V -> 25 V
- C23: value 10uF -> 2.2uF; LCSC (none) -> C19110; MPN (none) -> CL21B225KAFNNNE; Manufacturer (none) -> Samsung Electro-Mechanics; Placement (none) -> Local capacitor at U6.18 TVDD_IN; Status (none) -> PN7160 AN12988 local decoupling; selected stocked prototype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; Tolerance 20% -> 10%; Voltage 10 V -> 25 V
- C24: value 100nF -> 2.2uF; footprint Capacitor_SMD:C_0603_1608Metric -> Capacitor_SMD:C_0805_2012Metric; LCSC (none) -> C19110; MPN (none) -> CL21B225KAFNNNE; Manufacturer (none) -> Samsung Electro-Mechanics; Placement (none) -> Local capacitor at U6.22 TVDD; Status (none) -> PN7160 AN12988 local decoupling; selected stocked prototype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; Voltage 10 V -> 25 V
- C26: value 10pF START -> 12pF; MPN (none) -> CL10C120JB8NNNC; Manufacturer (none) -> Samsung Electro-Mechanics; Status (none) -> PROTOTYPE START: 12pF/15pF pair; tune carrier to -5..0ppm p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; Tolerance 10% -> 5%
- C27: value 10pF START -> 15pF; LCSC (none) -> C1644; MPN (none) -> CL10C150JB8NNNC; Manufacturer (none) -> Samsung Electro-Mechanics; Status (none) -> PROTOTYPE START: 12pF/15pF pair; tune carrier to -5..0ppm p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; Tolerance 10% -> 5%
- C28, C29: value TBD C_RX -> 1nF; footprint Capacitor_SMD:C_0603_1608Metric -> Capacitor_SMD:C_0805_2012Metric_Pad1.18x1.45mm_HandSolder; Dielectric C0G -> C0G/NP0; Status (none) -> PROTOTYPE START: validate with VNA / AGC / RF stress measur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; Tolerance 10% -> 5%; Voltage 50 V -> 100 V
- C30, C31: value TBD C_EMC -> 360pF; footprint Capacitor_SMD:C_0603_1608Metric -> Capacitor_SMD:C_0805_2012Metric_Pad1.18x1.45mm_HandSolder; Dielectric C0G -> C0G/NP0; Status (none) -> PROTOTYPE START: validate with VNA / AGC / RF stress measur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; Tolerance 10% -> 2%; Voltage 50 V -> 100 V
- C32, C33: value TBD C_SER -> 68pF; footprint Capacitor_SMD:C_0603_1608Metric -> Capacitor_SMD:C_0805_2012Metric_Pad1.18x1.45mm_HandSolder; Dielectric C0G -> C0G/NP0; Status (none) -> PROTOTYPE START: validate with VNA / AGC / RF stress measur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; Tolerance 10% -> 2%; Voltage 50 V -> 100 V
- C34, C35, C38, C39: value TBD C_TRIM -> DNP / TRIM; footprint Capacitor_SMD:C_0603_1608Metric -> Nucula_Project:C_0805_HandSolder_NoPaste; Dielectric C0G -> C0G/NP0; Status (none) -> DNP: fit equal pairs; 0.5-22pF typical fine trim; Tolerance 10% -> <=2% or +/-0.1pF for small trims; Voltage 50 V -> 100 V
- C36, C37: value TBD C_SHUNT -> 100pF; footprint Capacitor_SMD:C_0603_1608Metric -> Capacitor_SMD:C_0805_2012Metric_Pad1.18x1.45mm_HandSolder; Dielectric C0G -> C0G/NP0; Status (none) -> PROTOTYPE START: validate with VNA / AGC / RF stress measur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; Tolerance 10% -> 2%; Voltage 50 V -> 100 V
- L2, L3: value TBD L_EMC -> 150nH; footprint Nucula_Project:L_Coilcraft_0805HQ_2012Metric -> Nucula_Project:L_Coilcraft_0805HP; MPN (none) -> 0805HP-151XGRC; Manufacturer (none) -> Coilcraft; Status TUNE: high-Q RF inductor, >=0.5 A; self-resonance above ope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 -> PROTOTYPE: RF model included; 0.60A thermal reference, veri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; Tolerance (none) -> 2%
- R25, R26: value TBD R_RX -> 2.2k; footprint Resistor_SMD:R_0603_1608Metric -> Resistor_SMD:R_0805_2012Metric_Pad1.20x1.40mm_HandSolder; Rating 0.1 W -> 0.125 W; Status (none) -> PROTOTYPE: tune equal RX resistors for AGC 500-800 decimal
- R27, R28: value TBD R_DAMP -> 2.7R; footprint Resistor_SMD:R_0805_2012Metric -> Resistor_SMD:R_1206_3216Metric_Pad1.30x1.75mm_HandSolder; MPN (none) -> CRCW12062R70FKEAHP; Manufacturer (none) -> Vishay; Rating 0.25 W; RF loss/temperature to verify -> 0.75 W P70 only with Rth <=110 K/W; limit to 0.5W pending t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; Status (none) -> PROTOTYPE: Q about 20; also lift to measure bare antenna
- Y1: value 27.12MHz / CL TBD -> 27.12MHz / CL 10pF; footprint Crystal:Crystal_SMD_SeikoEpson_TSX3225-4Pin_3.2x2.5mm -> Nucula_Project:Crystal_NDK_NX2016SA_2.0x1.6mm; Candidate Family TSX-3225 27.1200MHz -> (none); Drive Level (none) -> 100 uW maximum; 10 uW typical; ESR (none) -> 100 ohm max, 25 ohm typical (NDK specification); LCSC (none) -> C3008209; Load Capacitance (none) -> 10 pF; MPN TBD load capacitance / ESR / drive grade -> NX2016SA-27.12MHZ-EXS00A-CS06346; Manufacturer Epson -> NDK; Status 27.12 MHz fixed; load capacitors require crystal selection -> SELECTED: NXP AN14518 reference; measure frequency/startup/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; Supply Status (none) -> JLCPCB C3008209: overseasStockCount 8896, purchasable 8533 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
Connections:
- net GND: now also C53.2, C54.1
- net NFC_TX1: now also R41.1; no longer L2.1
- net NFC_TX2: now also R42.1; no longer L3.1
- net RF_EMC_N: now also C54.2
- net RF_EMC_P: now also C53.1
- net at R28.2: now also A1.2 (LOOP_B)
- net at R27.2: now also A1.1 (LOOP_A)
- new net RF_DRV_N: L3.1, R42.2
- new net RF_DRV_P: L2.1, R41.2
Other:
- note added: "A1: 40x40 mm, 4T, 0.50/0.30 mm; estimated 1.56 uH. No GND tap. C34/C35, C38/C39, C53/C54: paired 0805 C0G tuning pads, DNP. Lift R41/R42 and R25/R26 to isolate RF tree for passive VNA tests. Lift R27/R28 for bare-coil measurement. NEVER power a connected VNA. Start TVDD <= 3.3 V; 20 ohm target trades field strength for current margin. See docs/nfc-antenna.md for calculations, layout rules and tun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"
- note added: "Pin 14 -> 18 + 22: internal TX-LDO output, not an external supply. Pin 31 -> 26 + 27: internal 1.8 V rail; decouple only. VSYS powers VBAT/VBAT2 and VDD_UP; VDD_PAD uses +3V3. ADR1:0 = 00 => 0x28. WKUP_REQ low; wake over I2C. VEN defaults low. DWL_REQ test access via its labelled net. ANT1/ANT2/VDHF unused: configure normal RF detection. Y1: NDK CS06346 27.12 MHz, CL 10pF; C26=12pF / C27=15pF. C2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"
- note added: "RF PROTOTYPE: 20 ohm differential target / measure before final tuning"
- note removed: "A1 pads 1/2 = coil ends; pad 3 = reference/shield ground. No center-tap assumption. Coil footprint is a placeholder. C34/C35/C38/C39 are optional parallel tuning pads (DNP). All other RF values are unselected; do not fabricate yet. Source: parts documentation/PN7160_schematic-3.pdf"
- note removed: "Pin 14 -> 18 + 22: internal TX-LDO output, not an external supply. Pin 31 -> 26 + 27: internal 1.8 V rail; decouple only. VSYS powers VBAT/VBAT2 and VDD_UP; VDD_PAD uses +3V3. ADR1:0 = 00 => 0x28. WKUP_REQ low; wake over I2C. VEN defaults low. DWL_REQ test access via its labelled net. ANT1/ANT2/VDHF unused: configure normal RF detection. 27.12 MHz crystal; confirm ESR, drive and load before order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"
- note removed: "RF values TBD: tune with the actual coil + final stackup"

Commit message: Prepare components and JLCPCB BOM for 10-board assembly
Parts:
- C26: LCSC (none) -> C38523
- C28, C29: LCSC (none) -> C162289; MPN (none) -> GRM2165C2A102JA01D; Manufacturer (none) -> Murata Electronics
- C30, C31: value 360pF -> 330pF; LCSC (none) -> C527075; MPN (none) -> CC0805FRNPO0BN331; Manufacturer (none) -> YAGEO; Status PROTOTYPE START: validate with VNA / AGC / RF stress measur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 -> PROTOTYPE: 330pF 1% + 33pF 5% in parallel = 363pF +/-1.364%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; Tolerance 2% -> 1%
- C32, C33: LCSC (none) -> C576904; MPN (none) -> CC0805FRNPO0BN680; Manufacturer (none) -> YAGEO; Tolerance 2% -> 1%
- C36, C37: LCSC (none) -> C527192; MPN (none) -> CC0805GRNPO0BN101; Manufacturer (none) -> YAGEO
- C53, C54: value TRIM -> 33pF; footprint Nucula_Project:C_0805_HandSolder_NoPaste -> Capacitor_SMD:C_0805_2012Metric_Pad1.18x1.45mm_HandSolder; LCSC (none) -> C309485; MPN (none) -> CC0805JRNPO0BN330; Manufacturer (none) -> YAGEO; Status DNP: EMC parallel trim; fit paired; replacing 360pF may be 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 -> PROTOTYPE: 330pF 1% + 33pF 5% in parallel = 363pF +/-1.364%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; Tolerance <=2% or +/-0.1pF for small trims -> 5%; now fitted
- L2, L3: LCSC (none) -> C20417049; Supply Status (none) -> 2026-09-20: JLCPCB C20417049 orderable 21; 10 boards requir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
- R21: LCSC (none) -> C25804; MPN (none) -> 0603WAF1002T5E; Manufacturer (none) -> UNI-ROYAL(Uniroyal Elec)
- R22, R23, R24: LCSC (none) -> C25803; MPN (none) -> 0603WAF1003T5E; Manufacturer (none) -> UNI-ROYAL(Uniroyal Elec)
- R25, R26: LCSC (none) -> C17520; MPN (none) -> 0805W8F2201T5E; Manufacturer (none) -> UNI-ROYAL(Uniroyal Elec)
- R27, R28: LCSC (none) -> C2079511; Manufacturer Vishay -> Vishay Intertech
- R29: LCSC (none) -> C21189; MPN (none) -> 0603WAF0000T5E; Manufacturer (none) -> UNI-ROYAL(Uniroyal Elec)
- R41, R42: LCSC (none) -> C96345; MPN (none) -> RC0805JR-070RL; Manufacturer (none) -> YAGEO; Rating 0.25 W; >=0.5A jumper current rating -> Jumper: 2 A rated; initial R <50 mOhm; 0.125 W package; Tolerance (none) -> Jumper
- U6: LCSC (none) -> C3303788; Manufacturer NXP -> NXP Semicon
- Y1: Supply Status JLCPCB C3008209: overseasStockCount 8896, purchasable 8533 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 -> 2026-09-20: JLCPCB C3008209 orderable 8538; in-stock assemb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
Other:
- note added: "A1: 40x40 mm, 4T, 0.50/0.30 mm; estimated 1.56 uH. No GND tap. C34/C35, C38/C39: paired 0805 C0G tuning pads, DNP. C30/C31 + C53/C54: 330 + 33 pF = 363 pF EMC shunt per leg. Lift R41/R42 and R25/R26 to isolate RF tree for passive VNA tests. Lift R27/R28 for bare-coil measurement. NEVER power a connected VNA. Start TVDD <= 3.3 V; 20 ohm target trades field strength for current margin. See docs/nfc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"
- note removed: "A1: 40x40 mm, 4T, 0.50/0.30 mm; estimated 1.56 uH. No GND tap. C34/C35, C38/C39, C53/C54: paired 0805 C0G tuning pads, DNP. Lift R41/R42 and R25/R26 to isolate RF tree for passive VNA tests. Lift R27/R28 for bare-coil measurement. NEVER power a connected VNA. Start TVDD <= 3.3 V; 20 ohm target trades field strength for current margin. See docs/nfc-antenna.md for calculations, layout rules and tun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"

Commit message: Add inside-feed NFC antenna and ESP antenna notch
Parts:
- A1: footprint Nucula_Project:NFC_PCB_Loop_40x40_4T_W0.50_S0.30 -> Nucula_Project:NFC_PCB_Loop_40x40_4T_W0.50_S0.30_InsideFeed; Status PROTOTYPE: 1.56uH estimated; measure RL/C before final tuni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 -> PROTOTYPE: inside-feed; 1.56uH unloaded estimate only; meas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
Changed lines of the file:
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@@
       )
     )
-    (property "Footprint" "Nucula_Project:NFC_PCB_Loop_40x40_4T_W0.50_S0.30"
+    (property "Footprint" "Nucula_Project:NFC_PCB_Loop_40x40_4T_W0.50_S0.30_InsideFeed"
       (at 391.16 91.44 0)
       (hide yes)
@@
       )
     )
-    (property "Status" "PROTOTYPE: 1.56uH estimated; measure RL/C before final tuning"
+    (property "Status" "PROTOTYPE: inside-feed; 1.56uH unloaded estimate only; measure with in-loop circuitry/ground"
       (at 391.16 96.52 0)
       (effects

Commit message: Complete four-layer PCB placement and routing
Preserve fixed placements and route all 91 nets with top-side components, symmetric NFC matching branches, antenna pour exclusions, and power/USB routing rules. Set front and back solder mask to black.

Add layout drawings, validation tooling and reports, and explicit NFC antenna net labels. Validation records zero DRC errors, zero unconnected items, zero schematic parity findings, and 23 passing layout checks; two existing silkscreen-edge warnings remain documented.
Connections:
- net Net-(A1-LOOP_B): now reaches A1.2 (LOOP_B), R28.2
- net Net-(A1-LOOP_A): now reaches A1.1 (LOOP_A), R27.2
Changed lines of the file:
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@@
+    )
+  )
+  (global_label "Net-(A1-LOOP_A)"
+    (shape bidirectional)
+    (at 368.3 73.66 0)
+    (effects
+      (font
+        (size 1.0 1.0)
+      )
+      (justify left)
+    )
+  )
+  (global_label "Net-(A1-LOOP_B)"
+    (shape bidirectional)
+    (at 368.3 119.38 0)
+    (effects
+      (font
+        (size 1.0 1.0)
+      )
+      (justify left)
     )
   )

Commit message: Qualify stocked parts and release October 9 production package
Replace four unavailable BOM lines, preserve rev-A NFC copper and placement, and include 792 simulation cases with fresh production validation. Remove superseded manufacturing packages so only the latest release remains.
Parts:
- C16, C18, C20, C25: LCSC C1591 -> C913912; MPN CL10B104KB8NNNC -> CL10B104KB8NNNL
- C28, C29: LCSC C162289 -> C326940; MPN GRM2165C2A102JA01D -> CC0805JRNPO0BN102; Manufacturer Murata Electronics -> YAGEO
- C36, C37: LCSC C527192 -> C464454; MPN CC0805GRNPO0BN101 -> 0805CG101F101NT; Manufacturer YAGEO -> FH (Guangdong Fenghua Advanced Tech); Tolerance 2% -> 1%
- L2, L3: footprint Nucula_Project:L_Coilcraft_0805HP -> Nucula_Project:L_Coilcraft_0805CS_RevALands; LCSC C20417049 -> C38190612; MPN 0805HP-151XGRC -> 0805CS-151XGLC; Status PROTOTYPE: RF model included; 0.60A thermal reference, veri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 -> RF substitute qualified by paired models; 0.40A DC thermal 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; Supply Status 2026-09-20: JLCPCB C20417049 orderable 21; 10 boards requir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 -> 2026-10-09: selected stocked substitute; see current JLC st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
Changed lines of the file:
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@@
       )
     )
-    (property "Datasheet" "https://product.samsungsem.com/mlcc/CL10B104KB8NNN.do"
+    (property "Datasheet" "https://product.samsungsem.com/cn/mlcc/CL10B104KB8NNN.do"
       (at 43.18 207.01 0)
       (effects
@@
       )
     )
-    (property "MPN" "CL10B104KB8NNNC"
+    (property "MPN" "CL10B104KB8NNNL"
       (at 43.18 207.01 0)
       (effects
@@
       )
     )
-    (property "LCSC" "C1591"
+    (property "LCSC" "C913912"
       (at 43.18 207.01 0)
       (effects
@@
       )
     )
-    (property "Datasheet" "https://product.samsungsem.com/mlcc/CL10B104KB8NNN.do"
+    (property "Datasheet" "https://product.samsungsem.com/cn/mlcc/CL10B104KB8NNN.do"
       (at 88.9 207.01 0)
       (effects
@@
       )
     )
-    (property "MPN" "CL10B104KB8NNNC"
+    (property "MPN" "CL10B104KB8NNNL"
       (at 88.9 207.01 0)
       (effects
@@
       )
     )
-    (property "LCSC" "C1591"
+    (property "LCSC" "C913912"
       (at 88.9 207.01 0)
       (effects
@@
       )
     )
-    (property "Datasheet" "https://product.samsungsem.com/mlcc/CL10B104KB8NNN.do"
+    (property "Datasheet" "https://product.samsungsem.com/cn/mlcc/CL10B104KB8NNN.do"
       (at 134.62 207.01 0)
       (effects
@@
       )
     )
-    (property "MPN" "CL10B104KB8NNNC"
+    (property "MPN" "CL10B104KB8NNNL"
       (at 134.62 207.01 0)
       (effects
@@
       )
     )
-    (property "LCSC" "C1591"
+    (property "LCSC" "C913912"
       (at 134.62 207.01 0)
       (effects
@@
       )
     )
-    (property "Datasheet" "https://product.samsungsem.com/mlcc/CL10B104KB8NNN.do"
+    (property "Datasheet" "https://product.samsungsem.com/cn/mlcc/CL10B104KB8NNN.do"
       (at 254 207.01 0)
       (effects
@@
       )
     )
-    (property "MPN" "CL10B104KB8NNNC"
+    (property "MPN" "CL10B104KB8NNNL"
       (at 254.0 207.01 0)
       (effects
@@
       )
     )
-    (property "LCSC" "C1591"
+    (property "LCSC" "C913912"
       (at 254.0 207.01 0)
       (effects
@@
       )
     )
-    (property "Footprint" "Nucula_Project:L_Coilcraft_0805HP"
+    (property "Footprint" "Nucula_Project:L_Coilcraft_0805CS_RevALands"
       (at 228.6 60.96 90)
       (effects
@@
       )
     )
-    (property "Datasheet" "https://www.coilcraft.com/en-us/products/rf/ceramic-core-chip-inductors/0805-(2012)/0805hp/0805hp-151/"
+    (property "Datasheet" "https://www.coilcraft.com/getmedia/dd5f20e4-1ff7-43df-8317-b693eb2dce3e/0805cs.pdf"
       (at 228.6 60.96 90)
       (effects
@@
       )
     )
-    (property "Status" "PROTOTYPE: RF model included; 0.60A thermal reference, verify actual RF heating"
+    (property "Status" "RF substitute qualified by paired models; 0.40A DC thermal reference; verify RF heating and read range on hardware"
       (at 228.6 60.96 90)
       (effects
@@
       )
     )
-    (property "MPN" "0805HP-151XGRC"
+    (property "MPN" "0805CS-151XGLC"
       (at 228.6 60.96 0)
       (effects
@@
       )
     )
-    (property "LCSC" "C20417049"
+    (property "LCSC" "C38190612"
       (at 228.6 60.96 0)
       (effects
@@
       )
     )
-    (property "Supply Status" "2026-09-20: JLCPCB C20417049 orderable 21; 10 boards require 20; secure stock before assembly"
+    (property "Supply Status" "2026-10-09: selected stocked substitute; see current JLC stock snapshot and qualification report"
       (at 228.6 60.96 0)
       (effects
@@
       )
     )
-    (property "Footprint" "Nucula_Project:L_Coilcraft_0805HP"
+    (property "Footprint" "Nucula_Project:L_Coilcraft_0805CS_RevALands"
       (at 228.6 132.08 90)
       (effects
@@
       )
     )
-    (property "Datasheet" "https://www.coilcraft.com/en-us/products/rf/ceramic-core-chip-inductors/0805-(2012)/0805hp/0805hp-151/"
+    (property "Datasheet" "https://www.coilcraft.com/getmedia/dd5f20e4-1ff7-43df-8317-b693eb2dce3e/0805cs.pdf"
       (at 228.6 132.08 90)
       (effects
@@
       )
     )
-    (property "Status" "PROTOTYPE: RF model included; 0.60A thermal reference, verify actual RF heating"
+    (property "Status" "RF substitute qualified by paired models; 0.40A DC thermal reference; verify RF heating and read range on hardware"
       (at 228.6 132.08 90)
       (effects
@@
       )
     )
-    (property "MPN" "0805HP-151XGRC"
+    (property "MPN" "0805CS-151XGLC"
       (at 228.6 132.08 0)
       (effects
@@
       )
     )
-    (property "LCSC" "C20417049"
+    (property "LCSC" "C38190612"
       (at 228.6 132.08 0)
       (effects
@@
       )
     )
-    (property "Supply Status" "2026-09-20: JLCPCB C20417049 orderable 21; 10 boards require 20; secure stock before assembly"
+    (property "Supply Status" "2026-10-09: selected stocked substitute; see current JLC stock snapshot and qualification report"
       (at 228.6 132.08 0)
       (effects
@@
       )
     )
-    (property "Datasheet" "https://wmsc.lcsc.com/wmsc/upload/file/pdf/v2/lcsc/2005222139_YAGEO-CC0805GRNPO0BN101_C527192.pdf"
+    (property "Datasheet" "https://wmsc.lcsc.com/wmsc/upload/file/pdf/v2/lcsc/2304140030_FH--Guangdong-Fenghua-Advanced-Tech-0805CG101F101NT_C464454.pdf"
       (at 307.34 78.74 0)
       (effects
@@
       )
     )
-    (property "Tolerance" "2%"
+    (property "Tolerance" "1%"
       (at 307.34 78.74 0)
       (effects
@@
       )
     )
-    (property "Manufacturer" "YAGEO"
+    (property "Manufacturer" "FH (Guangdong Fenghua Advanced Tech)"
       (at 307.34 78.74 0)
       (effects
@@
       )
     )
-    (property "MPN" "CC0805GRNPO0BN101"
+    (property "MPN" "0805CG101F101NT"
       (at 307.34 78.74 0)
       (effects
@@
       )
     )
-    (property "LCSC" "C527192"
+    (property "LCSC" "C464454"
       (at 307.34 78.74 0)
       (effects
@@
       )
     )
-    (property "Datasheet" "https://wmsc.lcsc.com/wmsc/upload/file/pdf/v2/lcsc/2005222139_YAGEO-CC0805GRNPO0BN101_C527192.pdf"
+    (property "Datasheet" "https://wmsc.lcsc.com/wmsc/upload/file/pdf/v2/lcsc/2304140030_FH--Guangdong-Fenghua-Advanced-Tech-0805CG101F101NT_C464454.pdf"
       (at 307.34 114.3 0)
       (effects
@@
       )
     )
-    (property "Tolerance" "2%"
+    (property "Tolerance" "1%"
       (at 307.34 114.3 0)
       (effects
@@
       )
     )
-    (property "Manufacturer" "YAGEO"
+    (property "Manufacturer" "FH (Guangdong Fenghua Advanced Tech)"
       (at 307.34 114.3 0)
       (effects
@@
       )
     )
-    (property "MPN" "CC0805GRNPO0BN101"
+    (property "MPN" "0805CG101F101NT"
       (at 307.34 114.3 0)
       (effects
@@
       )
     )
-    (property "LCSC" "C527192"
+    (property "LCSC" "C464454"
       (at 307.34 114.3 0)
       (effects
@@
       )
     )
-    (property "Datasheet" "https://www.lcsc.com/datasheet/lcsc_datasheet_2304140030_Murata-Electronics-GRM2165C2A102JA01D_C162289.pdf"
+    (property "Datasheet" "https://wmsc.lcsc.com/wmsc/upload/file/pdf/v2/lcsc/1811151646_YAGEO-CC0805JRNPO0BN102_C326940.pdf"
       (at 220.98 40.64 90)
       (effects
@@
       )
     )
-    (property "Manufacturer" "Murata Electronics"
+    (property "Manufacturer" "YAGEO"
       (at 220.98 40.64 0)
       (effects
@@
       )
     )
-    (property "MPN" "GRM2165C2A102JA01D"
+    (property "MPN" "CC0805JRNPO0BN102"
       (at 220.98 40.64 0)
       (effects
@@
       )
     )
-    (property "LCSC" "C162289"
+    (property "LCSC" "C326940"
       (at 220.98 40.64 0)
       (effects
@@
       )
     )
-    (property "Datasheet" "https://www.lcsc.com/datasheet/lcsc_datasheet_2304140030_Murata-Electronics-GRM2165C2A102JA01D_C162289.pdf"
+    (property "Datasheet" "https://wmsc.lcsc.com/wmsc/upload/file/pdf/v2/lcsc/1811151646_YAGEO-CC0805JRNPO0BN102_C326940.pdf"
       (at 220.98 165.1 90)
       (effects
@@
       )
     )
-    (property "Manufacturer" "Murata Electronics"
+    (property "Manufacturer" "YAGEO"
       (at 220.98 165.1 0)
       (effects
@@
       )
     )
-    (property "MPN" "GRM2165C2A102JA01D"
+    (property "MPN" "CC0805JRNPO0BN102"
       (at 220.98 165.1 0)
       (effects
@@
       )
     )
-    (property "LCSC" "C162289"
+    (property "LCSC" "C326940"
       (at 220.98 165.1 0)
       (effects
