File: oled.kicad_sch (KiCad schematic)
At the start: 23 parts, among them Q3 IRLML6402, Q4 BSS138, Q5 BSS138, U7 AP3012KTR-E1

Commit message: Fix display pin order and record USB backfeed diagnosis
Reverse the mounted display-to-socket mapping while preserving connector
geometry, reroute the local fanout, and add physical contact regression checks.
Refresh electrical, routing, fabrication, simulation and export validation.

Preserve the annotated Rev-A bench measurements and probe guides. Record
the accepted U4 data-to-VBUS diagnosis and the decision to proceed without
pin-isolation rework. The backfeed hardware remedy remains unimplemented.
Parts:
- DS1: symbol Nucula_Project:SSD1309_COG_24 -> Nucula_Project:SSD1309_COG_24_ReversedSocket; Actual Flex 24 contacts per user and supplied CON24 schematic; NFP1309-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 -> 24 contacts per user; panel pin 1 at PCB-left / socket pad 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; Connector Mechanics FH12A top-contact, 0.30 mm flex, 0.50 mm pitch; same copper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 -> FH12A top-contact, 0.30 mm flex, 0.50 mm pitch; manufacture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; Footprint Status SELECTED: 24-way 0.50 mm top-contact socket; Hirose drawing EDC3-150555-51 sheet 1 lands verified; supplied CON24 electrical map retained -> SELECTED: 24-way 0.50 mm top-contact socket; Hirose drawing EDC3-150555-51 sheet 1 lands verified; display pin n maps to socket pad 25-n; panel pin 1 is PCB-left; Status Top-contact socket selected for user-confirmed ribbon orientation; DS1 BOM is socket only; display and keyboard modules excluded; final physical fit and panel operation need prototype verification -> Top-contact socket selected for user-confirmed ribbon orientation; DS1 BOM is socket only; display and keyboard modules excluded; panel pin 1 confirmed PCB-left on 2026-10-06; validate operation on corrected board
Connections:
- net +3V0: now also DS1.19 (BS1), DS1.20 (VDD); no longer DS1.5 (VDD), DS1.6 (BS1)
- net GND: now also DS1.13 (E_RD), DS1.14 (RW), DS1.15 (SA0_DC), DS1.22 (VSS), DS1.23 (VLSS), DS1.5 (D7), DS1.6 (D6), DS1.9 (D3); no longer DS1.10 (SA0_DC), DS1.11 (RW), DS1.12 (E_RD), DS1.16 (D3), DS1.19 (D6), DS1.2 (VLSS), DS1.20 (D7), DS1.3 (VSS)
- net I2C_SCL: now also DS1.12 (D0_SCL); no longer DS1.13 (D0_SCL)
- net I2C_SDA: now also DS1.10 (D2_SDA_OUT), DS1.11 (D1_SDA_IN); no longer DS1.14 (D1_SDA_IN), DS1.15 (D2_SDA_OUT)
- net OLED_12V5: now also DS1.2 (VOP_PANEL); no longer DS1.23 (VOP_PANEL)
- net OLED_IREF: now also DS1.4 (IREF); no longer DS1.21 (IREF)
- net OLED_RES_N: now also DS1.16 (~{RES}); no longer DS1.9 (~{RES})
- net OLED_VCOMH: now also DS1.3 (VCOMH); no longer DS1.22 (VCOMH)
Other:
- note added: "DS1 numbers = Hirose socket pads. Display pin n = 25 - socket pad. PCB component-side view: panel pin 1 LEFT, pin 24 RIGHT. Keep socket position/orientation; do not mirror the footprint."
- note added: "Panel contact numbers (NOT DS1 socket pads): 13=SCL; 14+15=SDA; 9=RES#; 23=VOP. 1/2/3/24=GND; 4=NC; 5/6=3.0V. DS1 pad = 25 - panel pin; FH12A-24S socket. NFP1309-02Y: 0.50mm pitch, 0.30mm flex. Mounted tip contacts face away from PCB. SSD1309 I2C 0x3C, shared pull-ups 3.0V."
- note removed: "24 contacts: supplied CON24 breakout schematic. 13=SCL; 14+15=SDA; 9=RES#; 23=VOP. 1/2/3/24=GND; 4=NC; 5/6=3.0V. DS1: FH12A-24S top-contact socket only. NFP1309-02Y: 0.50mm pitch, 0.30mm flex. Mounted tip contacts face away from PCB. SSD1309 I2C 0x3C, shared pull-ups 3.0V."
Changed lines of the file:
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@@
   )
   (symbol
-    (lib_id "Nucula_Project:SSD1309_COG_24")
+    (lib_id "Nucula_Project:SSD1309_COG_24_ReversedSocket")
     (at 345.44 88.9 0)
     (unit 1)
@@
       )
     )
-    (property "Footprint Status" "SELECTED: 24-way 0.50 mm top-contact socket; Hirose drawing EDC3-150555-51 sheet 1 lands verified; supplied CON24 electrical map retained"
+    (property "Footprint Status" "SELECTED: 24-way 0.50 mm top-contact socket; Hirose drawing EDC3-150555-51 sheet 1 lands verified; display pin n maps to socket pad 25-n; panel pin 1 is PCB-left"
       (at 345.44 88.9 0)
       (effects
@@
       )
     )
-    (property "Actual Flex" "24 contacts per user and supplied CON24 schematic; NFP1309-02Y ribbon marking; 0.50 mm pitch, 0.30 mm thick; mounted tip contacts face away from PCB"
+    (property "Actual Flex" "24 contacts per user; panel pin 1 at PCB-left / socket pad 24; NFP1309-02Y ribbon marking; 0.50 mm pitch, 0.30 mm thick; mounted tip contacts face away from PCB"
       (at 345.44 88.9 0)
       (effects
@@
       )
     )
-    (property "Status" "Top-contact socket selected for user-confirmed ribbon orientation; DS1 BOM is socket only; display and keyboard modules excluded; final physical fit and panel operation need prototype verification"
+    (property "Status" "Top-contact socket selected for user-confirmed ribbon orientation; DS1 BOM is socket only; display and keyboard modules excluded; panel pin 1 confirmed PCB-left on 2026-10-06; validate operation on corrected board"
       (at 345.44 88.9 0)
       (effects
@@
       )
     )
-    (property "Connector Mechanics" "FH12A top-contact, 0.30 mm flex, 0.50 mm pitch; same copper lands and pin order; larger body/latch checked in layout; open latch height about 3.6 mm"
+    (property "Connector Mechanics" "FH12A top-contact, 0.30 mm flex, 0.50 mm pitch; manufacturer pad numbering retained; display pin n to socket pad 25-n; larger body/latch checked in layout; open latch height about 3.6 mm"
       (at 345.44 88.9 0)
       (effects
@@
       )
     )
+    (pin "19"
+    )
+    (pin "18"
+    )
+    (pin "17"
+    )
+    (pin "16"
+    )
+    (pin "15"
+    )
+    (pin "14"
+    )
+    (pin "13"
+    )
+    (pin "12"
+    )
+    (pin "11"
+    )
+    (pin "10"
+    )
+    (pin "9"
+    )
+    (pin "8"
+    )
+    (pin "7"
+    )
     (pin "6"
     )
-    (pin "7"
-    )
-    (pin "8"
-    )
-    (pin "9"
-    )
-    (pin "10"
-    )
-    (pin "11"
-    )
-    (pin "12"
-    )
-    (pin "13"
-    )
-    (pin "14"
-    )
-    (pin "15"
-    )
-    (pin "16"
-    )
-    (pin "17"
-    )
-    (pin "18"
-    )
-    (pin "19"
+    (pin "5"
     )
     (pin "20"
     )
-    (pin "5"
+    (pin "2"
+    )
+    (pin "4"
+    )
+    (pin "3"
+    )
+    (pin "24"
     )
     (pin "23"
     )
+    (pin "22"
+    )
+    (pin "1"
+    )
     (pin "21"
-    )
-    (pin "22"
-    )
-    (pin "1"
-    )
-    (pin "2"
-    )
-    (pin "3"
-    )
-    (pin "24"
-    )
-    (pin "4"
     )
     (instances
@@
     )
   )
-  (text "24 contacts: supplied CON24 breakout schematic.\n13=SCL; 14+15=SDA; 9=RES#; 23=VOP.\n1/2/3/24=GND; 4=NC; 5/6=3.0V.\nDS1: FH12A-24S top-contact socket only.\nNFP1309-02Y: 0.50mm pitch, 0.30mm flex.\nMounted tip contacts face away from PCB.\nSSD1309 I2C 0x3C, shared pull-ups 3.0V."
+  (text "Panel contact numbers (NOT DS1 socket pads):\n13=SCL; 14+15=SDA; 9=RES#; 23=VOP.\n1/2/3/24=GND; 4=NC; 5/6=3.0V.\nDS1 pad = 25 - panel pin; FH12A-24S socket.\nNFP1309-02Y: 0.50mm pitch, 0.30mm flex.\nMounted tip contacts face away from PCB.\nSSD1309 I2C 0x3C, shared pull-ups 3.0V."
     (at 20.32 246.38 0)
     (effects
@@
   )
   (embedded_fonts no)
+  (text "DS1 numbers = Hirose socket pads. Display pin n = 25 - socket pad.\nPCB component-side view: panel pin 1 LEFT, pin 24 RIGHT.\nKeep socket position/orientation; do not mirror the footprint." (at 318.77 139.7 0) (effects (font (size 1.27 1.27)) (justify left)))
 )

Commit message: Qualify stocked parts and release October 9 production package
Replace four unavailable BOM lines, preserve rev-A NFC copper and placement, and include 792 simulation cases with fresh production validation. Remove superseded manufacturing packages so only the latest release remains.
Parts:
- C43, C45, C48: LCSC C1591 -> C913912; MPN CL10B104KB8NNNC -> CL10B104KB8NNNL
Changed lines of the file:
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@@
       )
     )
-    (property "Datasheet" "https://www.lcsc.com/datasheet/lcsc_datasheet_2304140030_Samsung-Electro-Mechanics-CL10B104KB8NNNC_C1591.pdf"
+    (property "Datasheet" "https://product.samsungsem.com/cn/mlcc/CL10B104KB8NNN.do"
       (at 312.42 157.48 0)
       (effects
@@
       )
     )
-    (property "MPN" "CL10B104KB8NNNC"
+    (property "MPN" "CL10B104KB8NNNL"
       (at 312.42 157.48 0)
       (effects
@@
       )
     )
-    (property "LCSC" "C1591"
+    (property "LCSC" "C913912"
       (at 312.42 157.48 0)
       (effects
@@
       )
     )
-    (property "Datasheet" "https://www.lcsc.com/datasheet/lcsc_datasheet_2304140030_Samsung-Electro-Mechanics-CL10B104KB8NNNC_C1591.pdf"
+    (property "Datasheet" "https://product.samsungsem.com/cn/mlcc/CL10B104KB8NNN.do"
       (at 353.06 157.48 0)
       (effects
@@
       )
     )
-    (property "MPN" "CL10B104KB8NNNC"
+    (property "MPN" "CL10B104KB8NNNL"
       (at 353.06 157.48 0)
       (effects
@@
       )
     )
-    (property "LCSC" "C1591"
+    (property "LCSC" "C913912"
       (at 353.06 157.48 0)
       (effects
@@
       )
     )
-    (property "Datasheet" "https://www.lcsc.com/datasheet/lcsc_datasheet_2304140030_Samsung-Electro-Mechanics-CL10B104KB8NNNC_C1591.pdf"
+    (property "Datasheet" "https://product.samsungsem.com/cn/mlcc/CL10B104KB8NNN.do"
       (at 116.84 198.12 0)
       (effects
@@
       )
     )
-    (property "MPN" "CL10B104KB8NNNC"
+    (property "MPN" "CL10B104KB8NNNL"
       (at 116.84 198.12 0)
       (effects
@@
       )
     )
-    (property "LCSC" "C1591"
+    (property "LCSC" "C913912"
       (at 116.84 198.12 0)
       (effects
