File: power-mcu.kicad_sch (KiCad schematic)
At the start: 47 parts, among them J1 USB4105-GF-A, J2 JST-PH / 1S Li-ion, Q1 IRLML6402, Q2 BSS138, SW1 RESET, SW2 BOOT, U1 TP4054-42-SOT235, U2 SY8089AAAC, U3 ESP32-C3-WROOM-02-N4, U4 USBLC6-2SC6, U5 TLV803EA30DCKR

Commit message: Add PCB NFC coil and refine prototype component selections
Integrate a reusable 40 mm four-turn antenna footprint, calculated matching
network, hand-solder tuning pads, and a fabrication-ready bare-coil coupon.
Archive RF calculations, simulation results, reference sources, and tuning
instructions.

Select the PN7160 crystal and supply capacitors using manufacturer guidance
and DC-bias data. Record the confirmed 26-contact OLED interface and dedicated
5 V / 1.5 A USB-C source, retaining the JST-PH battery connector and deferred
battery behavior. Update the BOM, schematic PDFs, and verification tools.

Validation: native KiCad ERC reports zero violations; all current schematic
hashes match the verification report. Coil geometry, coupon DRC, RF model,
and component calculation results are archived with the design.
Parts:
- C1, C2, C4: footprint Capacitor_SMD:C_0805_2012Metric -> Capacitor_SMD:C_1210_3225Metric; Dielectric X5R -> X7R; LCSC (none) -> C309062; MPN (none) -> CL32B226KAJNNNE; Manufacturer (none) -> Samsung Electro-Mechanics; Status (none) -> SELECTED: manufacturer DC-bias curve checked; retain exact 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; Tolerance 20% -> 10%; Voltage 10 V -> 25 V
- C5, C6, C9: footprint Capacitor_SMD:C_0805_2012Metric -> Capacitor_SMD:C_1206_3216Metric; LCSC (none) -> C12891; MPN (none) -> CL31A226KAHNNNE; Manufacturer (none) -> Samsung Electro-Mechanics; Status (none) -> SELECTED: manufacturer DC-bias curve checked; Tolerance 20% -> 10%; Voltage 10 V -> 25 V
- J2: Status (none) -> OPTIONAL BATTERY TEST: JST-PH 2.00 mm; pin 1 BAT+, pin 2 GN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
Other:
- note added: "CC1 / CC2: independent 5.1k Rd. No USB-PD. Route D+/D- as a 90 ohm differential pair. Place U4 at connector; R12/R13 at module. Prototype source: 5 V USB-C, at least 1.5 A. Approx. 1.10 A planning budget; test startup/inrush."
- note added: "OPTIONAL battery test; USB works with J2 empty. J2: JST-PH 2.0mm; pin 1 = BAT+; pin 2 = GND. 100mA charge; protected 1S / 4.2V pack required. Battery performance deferred; check polarity before use."
- note added: "USB PROTOTYPE: dedicated 5 V / >=1.5 A source. Battery runtime and low-battery changes deferred. Test inrush, load steps and diode temperature. C1/C2/C4: 22uF / 25V / 1210; bias curve checked. Reference: Olimex ESP32-C3-DevKit-Lipo Rev C. See docs/component-refinements.md for calculations."
- note added: "VOUT = 3.31 V; R6 / R7: 0.1% precision 500 mA rail design target; validate transients. Buck only: low battery causes dropout / reset. C5/C6: 22uF each, 1206 / 25V; bias curve checked."
- note removed: "CC1 / CC2: independent 5.1k Rd. No USB-PD. Route D+/D- as a 90 ohm differential pair. Place U4 at connector; R12/R13 at module. See design notes for USB current / inrush limits."
- note removed: "DRAFT / before PCB: Confirm protected battery and JST polarity. Validate USB current, inrush, suspend and ESD. Verify regulator layout, capacitor bias and load steps. Reference: Olimex ESP32-C3-DevKit-Lipo Rev C. See docs/power-design.md for sources and limits."
- note removed: "Protected 1S LiPo, ~400mAh (3.7V nom / 4.2V full). J2: JST-PH 2.0mm; pin 1 = BAT+; pin 2 = GND. 100mA charge = 0.25C at 400mAh; ~10mA termination. Confirm pack polarity and ratings; no cell-temp input."
- note removed: "VOUT = 3.31 V; R6 / R7: 0.1% precision 500 mA rail design target; validate transients. Buck only: low battery causes dropout / reset. C5 + C6: 44 uF nominal; verify DC-bias derating."

Commit message: Prepare components and JLCPCB BOM for 10-board assembly
Parts:
- C10, C11, C13, C14: LCSC (none) -> C1591; MPN (none) -> CL10B104KB8NNNC; Manufacturer (none) -> Samsung Electro-Mechanics; Voltage 16 V -> 50 V
- C12: LCSC (none) -> C29936; MPN (none) -> CL10B105KA8NNNC; Manufacturer (none) -> Samsung Electro-Mechanics; Voltage 16 V -> 25 V
- C3: LCSC (none) -> C1653; MPN (none) -> CL10C220JB8NNNC; Manufacturer (none) -> Samsung Electro-Mechanics; Tolerance 10% -> 5%; Voltage 16 V -> 50 V
- D1, D2: LCSC (none) -> C85098
- D3: LCSC (none) -> C2286; MPN (none) -> KT-0603R; Manufacturer (none) -> Hubei KENTO Elec
- J1: value USB4105-GF-A -> USB4105-GF-A-120; LCSC (none) -> C5184243; MPN USB4105-GF-A -> USB4105-GF-A-120; Manufacturer GCT -> Global Connector Technology; Mechanical Note (none) -> 1.20 mm shell stakes; common USB4105 XY PCB pattern; 1.6 mm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
- J2: LCSC (none) -> C131337
- L1: LCSC (none) -> C6980123
- Q1: LCSC (none) -> C2593; Manufacturer Infineon -> Infineon Technologies
- Q2: LCSC (none) -> C52895
- R1, R2: LCSC (none) -> C23186; MPN (none) -> 0603WAF5101T5E; Manufacturer (none) -> UNI-ROYAL(Uniroyal Elec)
- R10, R11, R3, R5, R8, R9: LCSC (none) -> C25804; MPN (none) -> 0603WAF1002T5E; Manufacturer (none) -> UNI-ROYAL(Uniroyal Elec)
- R12, R13: LCSC (none) -> C23345; MPN (none) -> 0603WAF220JT5E; Manufacturer (none) -> UNI-ROYAL(Uniroyal Elec)
- R14: LCSC (none) -> C22775; MPN (none) -> 0603WAF1000T5E; Manufacturer (none) -> UNI-ROYAL(Uniroyal Elec)
- R15, R16: LCSC (none) -> C23178; MPN (none) -> 0603WAF4703T5E; Manufacturer (none) -> UNI-ROYAL(Uniroyal Elec)
- R17, R18: LCSC (none) -> C25803; MPN (none) -> 0603WAF1003T5E; Manufacturer (none) -> UNI-ROYAL(Uniroyal Elec)
- R4: LCSC (none) -> C4190; MPN (none) -> 0603WAF2201T5E; Manufacturer (none) -> UNI-ROYAL(Uniroyal Elec)
- R6: LCSC (none) -> C861231; MPN (none) -> RT0603BRD07220KL; Manufacturer (none) -> YAGEO
- R7: LCSC (none) -> C861429; MPN (none) -> RT0603BRD0748K7L; Manufacturer (none) -> YAGEO
- SW1, SW2: LCSC (none) -> C231329; Manufacturer Omron -> Omron Electronics
- U1: value TP4054-42-SOT235 -> TP4054-42-SOT25R; symbol Nucula_Project:TP4054-42-SOT235 -> Nucula_Project:TP4054-42-SOT25R; LCSC (none) -> C32574; MPN TP4054-42-SOT235 -> TP4054-42-SOT25R; Manufacturer Top Power ASIC -> TOPPOWER(Nanjing Extension Microelectronics)
- U2: LCSC (none) -> C78988; Manufacturer Silergy -> Silergy Corp
- U3: LCSC (none) -> C2934560; Manufacturer Espressif -> Espressif Systems
- U4: LCSC (none) -> C7519
- U5: value TLV803EA30DCKR -> TLV803EA30DBZR; footprint Package_TO_SOT_SMD:SOT-323_SC-70 -> Package_TO_SOT_SMD:SOT-23; symbol Nucula_Project:TLV803EA30DCKR -> Nucula_Project:TLV803EA30DBZR; LCSC (none) -> C5218924; MPN TLV803EA30DCKR -> TLV803EA30DBZR

Commit message: add break-away mouse bite line
Parts:
- J2: footprint Connector_JST:JST_PH_B2B-PH-K_1x02_P2.00mm_Vertical -> Nucula_Project:JST_PH_B2B-PH-SM4-TB_1x02-1MP_P2.00mm_Vertical; LCSC C131337 -> C160352; MPN B2B-PH-K-S(LF)(SN) -> B2B-PH-SM4-TB(LF)(SN); Status OPTIONAL BATTERY TEST: JST-PH 2.00 mm; pin 1 BAT+, pin 2 GN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 -> OPTIONAL BATTERY TEST: SMT top-entry JST-PH 2.00 mm; pin 1 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
Changed lines of the file:
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@@
       )
     )
-    (property "Footprint" "Connector_JST:JST_PH_B2B-PH-K_1x02_P2.00mm_Vertical"
+    (property "Footprint" "Nucula_Project:JST_PH_B2B-PH-SM4-TB_1x02-1MP_P2.00mm_Vertical"
       (at 248.92 45.72 0)
       (effects
@@
       )
     )
-    (property "MPN" "B2B-PH-K-S(LF)(SN)"
+    (property "MPN" "B2B-PH-SM4-TB(LF)(SN)"
       (at 248.92 45.72 0)
       (effects
@@
       )
     )
-    (property "Status" "OPTIONAL BATTERY TEST: JST-PH 2.00 mm; pin 1 BAT+, pin 2 GND; USB operation does not require a battery"
+    (property "Status" "OPTIONAL BATTERY TEST: SMT top-entry JST-PH 2.00 mm; pin 1 BAT+, pin 2 GND; mounting tabs unconnected; USB operation does not require a battery"
       (at 248.92 45.72 0)
       (effects
@@
       )
     )
-    (property "LCSC" "C131337"
+    (property "LCSC" "C160352"
       (at 248.92 45.72 0)
       (effects

Commit message: Fix USB connector clearance and prepare JLCPCB manufacturing release
Trim the two outer USB4105 ground lands by 0.04 mm at the locating-hole end, raising nominal NPTH clearance to 0.2333 mm. Use a project-local footprint and enforce JLCPCB's 0.20 mm minimum.

Regenerate Gerbers, drills, assembly files, drawings and source/hash archives. Refresh stock and ten-board purchasing quantities; add native and independent geometry validation. Preserve all placement, routing, holes and the confirmed OLED interface.
Parts:
- J1: footprint Connector_USB:USB_C_Receptacle_GCT_USB4105-xx-A_16P_TopMnt_Horizontal -> Nucula_Project:USB_C_GCT_USB4105_16P_JLCPCB
Changed lines of the file:
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@@
       )
     )
-    (property "Footprint" "Connector_USB:USB_C_Receptacle_GCT_USB4105-xx-A_16P_TopMnt_Horizontal"
+    (property "Footprint" "Nucula_Project:USB_C_GCT_USB4105_16P_JLCPCB"
       (at 27.94 53.34 0)
       (effects

Commit message: Standardize PCB fabrication and repair routing
Use ordinary open vias and adapted connector lands, retain a 17.70 x 5.00 mm display-ribbon access area, and rebuild routing with substantial pad entries and continuous 45-degree trace joins.

Add independent routing-quality checks, refreshed validation and simulations, sourcing notes, and complete five-board manufacturing packages. Preserve the submitted JLCPCB r2 archive.

Validation: zero DRC errors, unconnected items or schematic-parity findings; six routing checks, 21 layout checks and 16 fabrication checks pass. All 261 scoped simulations complete without solver errors. Cosmetic warnings and USB advisories are documented.
Parts:
- J1: footprint Nucula_Project:USB_C_GCT_USB4105_16P_JLCPCB -> Nucula_Project:USB_C_GCT_USB4105_16P_Standard
- U3: footprint Nucula_Project:ESP32-C3-WROOM-02-N4 -> Nucula_Project:ESP32-C3-WROOM-02-N4_NoEPADSolder
Changed lines of the file:
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@@
       )
     )
-    (property "Footprint" "Nucula_Project:USB_C_GCT_USB4105_16P_JLCPCB"
+    (property "Footprint" "Nucula_Project:USB_C_GCT_USB4105_16P_Standard"
       (at 27.94 53.34 0)
       (effects
@@
       )
     )
-    (property "Footprint" "Nucula_Project:ESP32-C3-WROOM-02-N4"
+    (property "Footprint" "Nucula_Project:ESP32-C3-WROOM-02-N4_NoEPADSolder"
       (at 96.52 172.72 0)
       (effects

Commit message: Fix USB backfeed with ground-referenced protection and data isolation
Parts:
- removed C7, C8: DNP / USB tune, Capacitor_SMD:C_0603_1608Metric, symbol Device:C
- added C55: 100nF, Capacitor_SMD:C_0603_1608Metric, symbol Device:C
- added D5: TPD1E10B06DYAR, Diode_SMD:D_SOD-523, symbol Device:D_TVS
- added U10: TS3USB30EDGSR, Package_SO:TSSOP-10_3x3mm_P0.5mm, symbol Interface_USB:TS3USB30EDGSR
- R17, R18: value 100k -> 10k; LCSC C25803 -> C25804; MPN 0603WAF1003T5E -> 0603WAF1002T5E
- U4: value USBLC6-2SC6 -> TPD2E2U06QDCKRQ1; footprint Package_TO_SOT_SMD:SOT-23-6 -> Package_TO_SOT_SMD:SOT-323_SC-70; symbol Power_Protection:USBLC6-2SC6 -> Power_Protection:TPD2E2U06DCK; LCSC C7519 -> C915089; MPN USBLC6-2SC6 -> TPD2E2U06QDCKRQ1; Manufacturer STMicroelectronics -> Texas Instruments
Connections:
- net +3V3: now also C55.1, U10.10 (VCC)
- net GND: now also U4.3, C55.2, D5.2 (A2), U10.1 (S), U10.5 (GND); no longer U4.2 (GND)
- net USB_D+: now also U4.2, U10.4 (D+); no longer U4.3 (I/O2)
- net USB_D-: now also U10.6 (D-)
- net USB_PRESENT_N: now also U10.9 (~{OE})
- net VBUS: now also D5.1 (A1); no longer U4.5 (VBUS)
- net USB_ESD_D+ renamed USB_PHY_D+
- net USB_PHY_D+: now also U10.2 (D1+); no longer U4.4 (I/O2)
- net USB_ESD_D- renamed USB_PHY_D-
- net USB_PHY_D-: now also U10.8 (D1-); no longer U4.6 (I/O1)
- no-connect marks 3 -> 5
Other:
- note added: "CC1 / CC2: independent 5.1k Rd. No USB-PD. U4 clamps data to GND; D5 protects VBUS separately. No data-to-VBUS steering-diode connection. Place U4/D5 at connector; R12/R13 at module. Prototype source: 5 V USB-C, at least 1.5 A."
- note added: "U10: hardware USB attach gating (also active in ROM). OE high = both data lines disconnected; S tied low."
- note added: "VBAT_ADC = VBAT / 2, max ~2.15 V incl. tolerances. ADC1 GPIO0: use calibrated 11/12 dB attenuation. Divider load ~4.5 uA; allow >=120 ms to settle. USB_PRESENT_N: GPIO1 LOW when VBUS is present. U10 disconnects USB data when VBUS is absent. GPIO1 must remain an input; attach gating is hardware. Q2 isolates 5 V VBUS from the 3.3 V GPIO / OE net."
- note removed: "CC1 / CC2: independent 5.1k Rd. No USB-PD. Route D+/D- as a 90 ohm differential pair. Place U4 at connector; R12/R13 at module. Prototype source: 5 V USB-C, at least 1.5 A. Approx. 1.10 A planning budget; test startup/inrush."
- note removed: "VBAT_ADC = VBAT / 2, max ~2.15 V incl. tolerances. ADC1 GPIO0: use calibrated 11/12 dB attenuation. Divider load ~4.5 uA; allow >=120 ms to settle. USB_PRESENT_N: GPIO1 LOW when VBUS is present. Firmware must disable USB attach when VBUS is absent. Q2 isolates 5 V VBUS from the 3.3 V GPIO supply."

Commit message: Switch to ESP32-C3-MINI-1 with a flush antenna cutout
Replace WROOM-02 with MINI-1-H4X while preserving GPIO assignments and
4 MB flash. Resize the antenna notch and align the antenna tip with the
PCB edge; update the schematic, routing, footprint, model and BOM.

Include the current JST-SH battery connector and direct battery solder
pads, plus manufacturing archives and the new MINI prototype package.
Record ESP-IDF 5.4+ compatibility and the remaining physical validation.

Validation: zero ERC/DRC errors or unconnected nets; 17 MINI checks,
16 fabrication checks, six routing checks and 30 export checks pass.
The 261 scoped simulation cases completed without solver errors.
Parts:
- added J6: Battery wire pads, Nucula_Project:Battery_Lead_SolderPads_2x2.2x2.5mm_P3.4mm, symbol Connector_Generic:Conn_01x02
- J2: value JST-PH / 1S Li-ion -> JST-SH / 1S Li-ion; footprint Nucula_Project:JST_PH_B2B-PH-SM4-TB_1x02-1MP_P2.00mm_Vertical -> Nucula_Project:JST_SH_SM02B-SRSS-TB_1x02-1MP_P1.00mm_Horizontal; LCSC C160352 -> C160402; MPN B2B-PH-SM4-TB(LF)(SN) -> SM02B-SRSS-TB(LF)(SN); Status OPTIONAL BATTERY TEST: SMT top-entry JST-PH 2.00 mm; pin 1 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 -> OPTIONAL BATTERY TEST: SMT SIDE-ENTRY JST-SH 1.00 mm; 2.95 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
- U3: value ESP32-C3-WROOM-02-N4 -> ESP32-C3-MINI-1-H4X; footprint Nucula_Project:ESP32-C3-WROOM-02-N4_NoEPADSolder -> Nucula_Project:ESP32-C3-MINI-1-H4X_NoEPADSolder; symbol Nucula_Project:ESP32-C3-WROOM-02-N4 -> Nucula_Project:ESP32-C3-MINI-1-H4X; LCSC C2934560 -> C41349510; MPN ESP32-C3-WROOM-02-N4 -> ESP32-C3-MINI-1-H4X
Connections:
- net +3V3: now also U3.3 (3V3); no longer U3.1 (3V3)
- net BOOT_N: now also U3.23 (IO9); no longer U3.8 (IO9)
- net ESP_EN: now also U3.8 (EN); no longer U3.2 (EN)
- net GND: now also U3.1 (GND), U3.11 (GND), U3.14 (GND), U3.2 (GND), U3.36 (GND), U3.37 (GND), U3.38 (GND), U3.39 (GND), U3.40 (GND), U3.41 (GND), U3.42 (GND), U3.43 (GND), U3.44 (GND), U3.45 (GND), U3.46 (GND), U3.47 (GND), U3.48 (GND), U3.49 (GND), U3.50 (GND), U3.51 (GND), U3.52 (GND), U3.53 (GND), J6.2 (Pin_2); no longer U3.19 (GND), U3.9 (GND)
- net I2C_SCL: now also U3.19 (IO5); no longer U3.4 (IO5)
- net I2C_SDA: now also U3.18 (IO4); no longer U3.3 (IO4)
- net KEY_INT_N: now also U3.30 (IO20/RXD); no longer U3.11 (IO20/RXD)
- net NFC_IRQ: now also U3.20 (IO6); no longer U3.5 (IO6)
- net NFC_VEN: now also U3.21 (IO7); no longer U3.6 (IO7)
- net OLED_PWR_EN: now also U3.6 (IO3); no longer U3.15 (IO3)
- net OLED_RESET: now also U3.16 (IO10); no longer U3.10 (IO10)
- net STRAP_GPIO2: now also U3.5 (IO2); no longer U3.16 (IO2)
- net STRAP_GPIO8: now also U3.22 (IO8); no longer U3.7 (IO8)
- net USB_PRESENT_N: now also U3.13 (IO1); no longer U3.17 (IO1)
- net VBAT: now also J6.1 (Pin_1)
- net VBAT_ADC: now also U3.12 (IO0); no longer U3.18 (IO0)
- net at R13.2: now also U3.27 (IO19); no longer U3.14 (IO19)
- net at R12.2: now also U3.26 (IO18); no longer U3.13 (IO18)
Other:
- note added: "OPTIONAL battery test; USB works without a battery. J2: JST-SH side entry OR J6: direct wire solder pads. Both: pin 1 = BAT+; pin 2 = GND. Use ONE battery connection. 100mA charge; protected 1S / 4.2V pack; check polarity."
- note removed: "OPTIONAL battery test; USB works with J2 empty. J2: JST-PH 2.0mm; pin 1 = BAT+; pin 2 = GND. 100mA charge; protected 1S / 4.2V pack required. Battery performance deferred; check polarity before use."

Commit message: Qualify stocked parts and release October 9 production package
Replace four unavailable BOM lines, preserve rev-A NFC copper and placement, and include 792 simulation cases with fresh production validation. Remove superseded manufacturing packages so only the latest release remains.
Parts:
- C10, C11, C13, C14, C55: LCSC C1591 -> C913912; MPN CL10B104KB8NNNC -> CL10B104KB8NNNL
Changed lines of the file:
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@@
       )
     )
-    (property "Datasheet" "https://www.lcsc.com/datasheet/lcsc_datasheet_2304140030_Samsung-Electro-Mechanics-CL10B104KB8NNNC_C1591.pdf"
+    (property "Datasheet" "https://product.samsungsem.com/cn/mlcc/CL10B104KB8NNN.do"
       (at 127 71.12 0)
       (effects
@@
       )
     )
-    (property "MPN" "CL10B104KB8NNNC"
+    (property "MPN" "CL10B104KB8NNNL"
       (at 127 71.12 0)
       (effects
@@
       )
     )
-    (property "LCSC" "C1591"
+    (property "LCSC" "C913912"
       (at 127 71.12 0)
       (effects
@@
       )
     )
-    (property "Datasheet" "https://www.lcsc.com/datasheet/lcsc_datasheet_2304140030_Samsung-Electro-Mechanics-CL10B104KB8NNNC_C1591.pdf"
+    (property "Datasheet" "https://product.samsungsem.com/cn/mlcc/CL10B104KB8NNN.do"
       (at 142.24 203.2 0)
       (effects
@@
       )
     )
-    (property "MPN" "CL10B104KB8NNNC"
+    (property "MPN" "CL10B104KB8NNNL"
       (at 142.24 203.2 0)
       (effects
@@
       )
     )
-    (property "LCSC" "C1591"
+    (property "LCSC" "C913912"
       (at 142.24 203.2 0)
       (effects
@@
       )
     )
-    (property "Datasheet" "https://www.lcsc.com/datasheet/lcsc_datasheet_2304140030_Samsung-Electro-Mechanics-CL10B104KB8NNNC_C1591.pdf"
+    (property "Datasheet" "https://product.samsungsem.com/cn/mlcc/CL10B104KB8NNN.do"
       (at 175.26 152.4 0)
       (effects
@@
       )
     )
-    (property "MPN" "CL10B104KB8NNNC"
+    (property "MPN" "CL10B104KB8NNNL"
       (at 175.26 152.4 0)
       (effects
@@
       )
     )
-    (property "LCSC" "C1591"
+    (property "LCSC" "C913912"
       (at 175.26 152.4 0)
       (effects
@@
       )
     )
-    (property "Datasheet" "https://www.lcsc.com/datasheet/lcsc_datasheet_2304140030_Samsung-Electro-Mechanics-CL10B104KB8NNNC_C1591.pdf"
+    (property "Datasheet" "https://product.samsungsem.com/cn/mlcc/CL10B104KB8NNN.do"
       (at 309.88 177.8 0)
       (effects
@@
       )
     )
-    (property "MPN" "CL10B104KB8NNNC"
+    (property "MPN" "CL10B104KB8NNNL"
       (at 309.88 177.8 0)
       (effects
@@
       )
     )
-    (property "LCSC" "C1591"
+    (property "LCSC" "C913912"
       (at 309.88 177.8 0)
       (effects
@@
       )
     )
-    (property "Datasheet" "https://www.lcsc.com/datasheet/lcsc_datasheet_2304140030_Samsung-Electro-Mechanics-CL10B104KB8NNNC_C1591.pdf"
+    (property "Datasheet" "https://product.samsungsem.com/cn/mlcc/CL10B104KB8NNN.do"
       (at 246.38 107.95 0)
       (effects
@@
       )
     )
-    (property "MPN" "CL10B104KB8NNNC"
+    (property "MPN" "CL10B104KB8NNNL"
       (at 246.38 107.95 0)
       (effects
@@
       )
     )
-    (property "LCSC" "C1591"
+    (property "LCSC" "C913912"
       (at 246.38 107.95 0)
       (effects
